File: _autosave-OSU-keyboard-V1.kicad_sch (KiCad schematic)
At the start: 21 parts, among them J1 AVR-ISP-6, SW1 SW_Push_Dual, U1 ATmega32U4-A, U2 PRTR5V0U2X, Y1 16MHz

Commit message: Schematic finish
Just about to enter to PCB
Parts:
- added D1, D2, D3, D4: D_Small, symbol Device:D_Small
- added MX1, MX2, MX3, MX4: MX-NoLED, Package_TO_SOT_SMD:SOT-23W_Handsoldering, symbol MX_Alps_Hybrid:MX-NoLED
- R1: value 10K -> 10k
Connections:
- net +5V: now also U1.7 (VBUS)
- net GND: now also U2.1 (GND)
- net VCC: now also U2.4 (VCC)
- net at R3.1, USB1.5 (DN2), USB1.7 (DN1): now also U2.3 (IO2)
- net at R4.1, USB1.6 (DP1), USB1.8 (DP2): now also U2.2 (IO1)
- net COL0: now reaches U1.28 (PB4)
- net COL0: now also MX1.1 (COL), MX4.1 (COL)
- net COL1: now reaches U1.29 (PB5)
- net COL1: now also MX2.1 (COL)
- net COL2: now reaches U1.30 (PB6)
- net COL2: now also MX3.1 (COL)
- net ROW0: now reaches U1.31 (PC6)
- net ROW0: now also D1.1 (K), D2.1 (K), D3.1 (K)
- net ROW1: now reaches U1.32 (PC7)
- net ROW1: now also D4.1 (K)
- new net: D4.2 (A), MX4.2 (ROW)
- new net: D1.2 (A), MX1.2 (ROW)
- new net: D2.2 (A), MX2.2 (ROW)
- new net: D3.2 (A), MX3.2 (ROW)
- no-connect marks 5 -> 22
Other:
- moved on the sheet: C1, C2, C3, C4, C5, C6, C7, C8, F1, J1, R1, R2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
